File: audio.kicad_sch (KiCad schematic)
At the start: 13 parts, among them J3 SJ-3523-SMT-TR, U6 PCM5102APWR, U7 TPA6132A2RTER

Commit message: work on pcb
Parts:
- J3: footprint SJ-3523-SMT-TR:CUI_SJ-3523-SMT-TR -> audio-jack:CUI_SJ-3523-SMT-TR
- U6: footprint PCM5102APWR:SOP65P640X120-20N -> dac:SOP65P640X120-20N
- U7: footprint TPA6132A2RTER:QFN50P300X300X80-16N -> amp:QFN50P300X300X80-16N
Connections:
- net IO_DAC_SCK is gone; now on net GND: U6.12 (SCK)
Changed lines of the file:
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@@
-		)
-	)
-	(hierarchical_label "IO_DAC_SCK"
-		(shape input)
-		(at 69.85 54.61 180)
-		(effects
-			(font
-				(size 1.27 1.27)
-			)
-			(justify right)
 		)
 	)
@@
 	)
 	(symbol
+		(lib_id "power:GND")
+		(at 69.85 54.61 270)
+		(unit 1)
+		(body_style 1)
+		(exclude_from_sim no)
+		(in_bom yes)
+		(on_board yes)
+		(in_pos_files yes)
+		(dnp no)
+		(fields_autoplaced yes)
+		(property "Reference" "#PWR063"
+			(at 63.5 54.61 0)
+			(hide yes)
+			(show_name no)
+			(do_not_autoplace no)
+			(effects
+				(font
+					(size 1.27 1.27)
+				)
+			)
+		)
+		(property "Value" "GND"
+			(at 66.04 54.6099 90)
+			(show_name no)
+			(do_not_autoplace no)
+			(effects
+				(font
+					(size 1.27 1.27)
+				)
+				(justify right)
+			)
+		)
+		(property "Footprint" ""
+			(at 69.85 54.61 0)
+			(hide yes)
+			(show_name no)
+			(do_not_autoplace no)
+			(effects
+				(font
+					(size 1.27 1.27)
+				)
+			)
+		)
+		(property "Datasheet" ""
+			(at 69.85 54.61 0)
+			(hide yes)
+			(show_name no)
+			(do_not_autoplace no)
+			(effects
+				(font
+					(size 1.27 1.27)
+				)
+			)
+		)
+		(property "Description" "Power symbol creates a global label with name \"GND\" , ground"
+			(at 69.85 54.61 0)
+			(hide yes)
+			(show_name no)
+			(do_not_autoplace no)
+			(effects
+				(font
+					(size 1.27 1.27)
+				)
+			)
+		)
+		(pin "1"
+		)
+		(instances
+			(project "e507"
+				(path "/acf7fdfc-08c7-4b01-88b5-5cee2f49d989/f3ecc11f-918d-4403-b589-59b01044df1d"
+					(reference "#PWR063")
+					(unit 1)
+				)
+			)
+		)
+	)
+	(symbol
 		(lib_id "power:+3V3")
 		(at 40.64 99.06 0)
@@
 			)
 		)
-		(property "Footprint" "TPA6132A2RTER:QFN50P300X300X80-16N"
+		(property "Footprint" "amp:QFN50P300X300X80-16N"
 			(at 87.63 151.13 0)
 			(hide yes)
@@
 			)
 		)
-		(property "Footprint" "PCM5102APWR:SOP65P640X120-20N"
+		(property "Footprint" "dac:SOP65P640X120-20N"
 			(at 87.63 62.23 0)
 			(hide yes)
@@
 			)
 		)
-		(property "Footprint" "SJ-3523-SMT-TR:CUI_SJ-3523-SMT-TR"
+		(property "Footprint" "audio-jack:CUI_SJ-3523-SMT-TR"
 			(at 262.89 62.23 0)
 			(hide yes)
