File: audio.kicad_sch (KiCad schematic)
At the start: 13 parts, among them J3 SJ-3523-SMT-TR, U6 PCM5102APWR, U7 TPA6132A2RTER

Commit message: fucker
Parts:
- added C22, C23, C28, C29: 1μF, symbol Device:C_Small
- added C24, C25: 2.2μF, symbol Device:C_Small
- added C26, C27: 2.2nF, symbol Device:C_Small
- added R18: 10K, symbol Device:R_Small
- added R19, R20: 470Ω, symbol Device:R_Small
- C12, C16, C18, C21: value 0.1uF -> 0.1μF
- C13, C17, C19, C20: value 10uF -> 10μF
- C14, C15: value 2.2uF -> 2.2μF
- J3: footprint audio-jack:CUI_SJ-3523-SMT-TR -> SJ-3523-SMT-TR:CUI_SJ-3523-SMT-TR
- U6: footprint dac:SOP65P640X120-20N -> PCM5102APWR:SOP65P640X120-20N
- U7: footprint amp:QFN50P300X300X80-16N -> TPA6132A2RTER:QFN50P300X300X80-16N
Connections:
- net GND: now also U7.10 (PGND), U7.17 (EP), U7.2 (INL+), U7.3 (INR+), C23.2, C24.1, C25.1, R18.1; no longer C12.1, C13.2, C14.2, C16.1, C17.2, U6.12 (SCK), U6.3 (CPGND), U6.9 (AGND)
- net at U7.1 (INL-): now also C28.2
- net at U7.11 (CPP): now also C22.2
- net at U7.12 (HPVDD): now also C24.2
- net IO_AMP_EN: now reaches U7.13 (EN)
- net IO_AMP_EN: now also R18.2
- net VSYS: now reaches U7.14 (VDD)
- net VSYS: now also C25.2
- net GNDA: now reaches U7.15 (SGND)
- net GNDA: now also C12.1, C13.2, C14.2, C16.1, C17.2, J3.1 (SLEEVE), U6.3 (CPGND), U6.9 (AGND), C26.1, C27.2
- net at U7.16 (OUTL): now also J3.2 (TIP)
- net at U7.4 (INR-): now also C29.2
- net at U7.5 (OUTR): now also J3.3 (RING)
- net at U7.8 (HPVSS): now also C23.1
- net at U7.9 (CPN): now also C22.1
- net at U6.6 (OUTL): now also R19.1
- net at U6.7 (OUTR): now also R20.1
- new net DAC_L: C26.2, C28.1, R19.2
- new net DAC_R: C27.1, C29.1, R20.2
- new net IO_DAC_SCK: U6.12 (SCK)
Other:
- moved on the sheet: J3, U7

Commit message: Finish? schematic
Parts:
- J3: footprint SJ-3523-SMT-TR:CUI_SJ-3523-SMT-TR -> audio-jack:CUI_SJ-3523-SMT-TR
- U6: footprint PCM5102APWR:SOP65P640X120-20N -> dac:SOP65P640X120-20N
- U7: footprint TPA6132A2RTER:QFN50P300X300X80-16N -> amp:QFN50P300X300X80-16N
Connections:
- net IO_DAC_SCK is gone; now on net GND: U6.12 (SCK)
- net GND: now also C23.1, U7.7 (G1); no longer C23.2
- net VSYS: now also U7.6 (G0)
- net at U7.8 (HPVSS): now also C23.2; no longer C23.1
Other:
- moved on the sheet: C23

Commit message: holy routing
Parts:
- C12, C13, C14, C15, C16, C17, C18, C19, C20, C21, C22, C23, C24, C25, C26, C27, C28, C29: footprint (none) -> Capacitor_SMD:C_0201_0603Metric
- R18, R19, R20: footprint (none) -> Resistor_SMD:R_0201_0603Metric
Connections:
- net VSYS is gone; now on net +3V3_AUDIO: C25.2, U7.14 (VDD), U7.6 (G0)
- net GND: no longer C23.1, C24.1, C25.1, R18.1, U7.10 (PGND), U7.17 (EP), U7.2 (INL+), U7.3 (INR+), U7.7 (G1)
- net GNDA: now also C23.1, C24.1, C25.1, R18.1, U7.10 (PGND), U7.17 (EP), U7.2 (INL+), U7.3 (INR+), U7.7 (G1)
Other:
- moved on the sheet: R18

Commit message: switch to stm32, wire audio section
Parts:
- C12, C13, C14, C15, C16, C17, C18, C19, C20, C21, C22, C23, C24, C25, C26, C27, C28, C29: footprint Capacitor_SMD:C_0201_0603Metric -> Capacitor_SMD:C_0402_1005Metric
- R18, R19, R20: footprint Resistor_SMD:R_0201_0603Metric -> Resistor_SMD:R_0402_1005Metric
Connections:
- net DAC_L: now also C29.1; no longer C28.1
- net DAC_R: now also C28.1; no longer C29.1
- net GND: no longer U6.10 (DEMP)
- net GNDA: now also U6.10 (DEMP)
Changed lines of the file:
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@@
 		)
 	)
-	(label "DAC_R"
+	(label "DAC_L"
 		(at 46.99 144.78 180)
 		(effects
@@
 		)
 	)
-	(label "DAC_L"
+	(label "DAC_R"
 		(at 46.99 140.97 180)
 		(effects
@@
 			)
 		)
-		(property "Footprint" "Resistor_SMD:R_0201_0603Metric"
+		(property "Footprint" "Resistor_SMD:R_0402_1005Metric"
 			(at 41.91 157.48 0)
 			(hide yes)
@@
 			)
 		)
-		(property "Footprint" "Capacitor_SMD:C_0201_0603Metric"
+		(property "Footprint" "Capacitor_SMD:C_0402_1005Metric"
 			(at 111.76 80.01 0)
 			(hide yes)
@@
 			)
 		)
-		(property "Footprint" "Capacitor_SMD:C_0201_0603Metric"
+		(property "Footprint" "Capacitor_SMD:C_0402_1005Metric"
 			(at 124.46 85.09 0)
 			(hide yes)
@@
 			)
 		)
-		(property "Footprint" "Capacitor_SMD:C_0201_0603Metric"
+		(property "Footprint" "Capacitor_SMD:C_0402_1005Metric"
 			(at 67.31 123.19 0)
 			(hide yes)
@@
 			)
 		)
-		(property "Footprint" "Capacitor_SMD:C_0201_0603Metric"
+		(property "Footprint" "Capacitor_SMD:C_0402_1005Metric"
 			(at 45.72 86.36 0)
 			(hide yes)
@@
 			)
 		)
-		(property "Footprint" "Capacitor_SMD:C_0201_0603Metric"
+		(property "Footprint" "Capacitor_SMD:C_0402_1005Metric"
 			(at 45.72 93.98 0)
 			(hide yes)
@@
 			)
 		)
-		(property "Footprint" "Resistor_SMD:R_0201_0603Metric"
+		(property "Footprint" "Resistor_SMD:R_0402_1005Metric"
 			(at 146.05 64.77 0)
 			(hide yes)
@@
 			)
 		)
-		(property "Footprint" "Capacitor_SMD:C_0201_0603Metric"
+		(property "Footprint" "Capacitor_SMD:C_0402_1005Metric"
 			(at 55.88 127 0)
 			(hide yes)
@@
 			)
 		)
-		(property "Footprint" "Capacitor_SMD:C_0201_0603Metric"
+		(property "Footprint" "Capacitor_SMD:C_0402_1005Metric"
 			(at 154.94 71.12 0)
 			(hide yes)
@@
 			)
 		)
-		(property "Value" "GND"
+		(property "Value" "GNDA"
 			(at 66.04 74.9299 90)
 			(show_name no)
@@
 			)
 		)
-		(property "Footprint" "Capacitor_SMD:C_0201_0603Metric"
+		(property "Footprint" "Capacitor_SMD:C_0402_1005Metric"
 			(at 124.46 52.07 0)
 			(hide yes)
@@
 			)
 		)
-		(property "Footprint" "Capacitor_SMD:C_0201_0603Metric"
+		(property "Footprint" "Capacitor_SMD:C_0402_1005Metric"
 			(at 58.42 93.98 0)
 			(hide yes)
@@
 			)
 		)
-		(property "Footprint" "Capacitor_SMD:C_0201_0603Metric"
+		(property "Footprint" "Capacitor_SMD:C_0402_1005Metric"
 			(at 57.15 166.37 0)
 			(hide yes)
@@
 			)
 		)
-		(property "Footprint" "Capacitor_SMD:C_0201_0603Metric"
+		(property "Footprint" "Capacitor_SMD:C_0402_1005Metric"
 			(at 52.07 140.97 0)
 			(hide yes)
@@
 			)
 		)
-		(property "Footprint" "Capacitor_SMD:C_0201_0603Metric"
+		(property "Footprint" "Capacitor_SMD:C_0402_1005Metric"
 			(at 58.42 86.36 0)
 			(hide yes)
@@
 			)
 		)
-		(property "Footprint" "Resistor_SMD:R_0201_0603Metric"
+		(property "Footprint" "Resistor_SMD:R_0402_1005Metric"
 			(at 146.05 67.31 0)
 			(hide yes)
@@
 			)
 		)
-		(property "Footprint" "Capacitor_SMD:C_0201_0603Metric"
+		(property "Footprint" "Capacitor_SMD:C_0402_1005Metric"
 			(at 111.76 85.09 0)
 			(hide yes)
@@
 			)
 		)
-		(property "Footprint" "Capacitor_SMD:C_0201_0603Metric"
+		(property "Footprint" "Capacitor_SMD:C_0402_1005Metric"
 			(at 62.23 135.89 0)
 			(hide yes)
@@
 			)
 		)
-		(property "Footprint" "Capacitor_SMD:C_0201_0603Metric"
+		(property "Footprint" "Capacitor_SMD:C_0402_1005Metric"
 			(at 111.76 71.12 0)
 			(hide yes)
@@
 			)
 		)
-		(property "Footprint" "Capacitor_SMD:C_0201_0603Metric"
+		(property "Footprint" "Capacitor_SMD:C_0402_1005Metric"
 			(at 52.07 144.78 0)
 			(hide yes)
@@
 			)
 		)
-		(property "Footprint" "Capacitor_SMD:C_0201_0603Metric"
+		(property "Footprint" "Capacitor_SMD:C_0402_1005Metric"
 			(at 111.76 52.07 0)
 			(hide yes)
@@
 			)
 		)
-		(property "Footprint" "Capacitor_SMD:C_0201_0603Metric"
+		(property "Footprint" "Capacitor_SMD:C_0402_1005Metric"
 			(at 154.94 60.96 0)
 			(hide yes)

Commit message: assign some dac caps
Parts:
- C12, C16, C18, C21: LCSC Part # (none) -> C307331; Part # (none) -> CL05B104KB54PNC
- C13, C17, C19, C20: LCSC Part # (none) -> C15525; Part # (none) -> CL05A106MQ5NUNC
- U6: LCSC Part # (none) -> C107671; Part # (none) -> PCM5102APWR
Changed lines of the file:
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@@
 			)
 		)
-		(property "LCSC Part #" ""
+		(property "LCSC Part #" "C15525"
 			(at 124.46 85.09 0)
 			(hide yes)
@@
 			)
 		)
-		(property "Part #" ""
+		(property "Part #" "CL05A106MQ5NUNC"
 			(at 124.46 85.09 0)
 			(hide yes)
@@
 			)
 		)
-		(property "LCSC Part #" ""
+		(property "LCSC Part #" "C107671"
 			(at 87.63 62.23 0)
 			(hide yes)
@@
 			)
 		)
-		(property "Part #" ""
+		(property "Part #" "PCM5102APWR"
 			(at 87.63 62.23 0)
 			(hide yes)
@@
 			)
 		)
-		(property "LCSC Part #" ""
+		(property "LCSC Part #" "C15525"
 			(at 45.72 86.36 0)
 			(hide yes)
@@
 			)
 		)
-		(property "Part #" ""
+		(property "Part #" "CL05A106MQ5NUNC"
 			(at 45.72 86.36 0)
 			(hide yes)
@@
 			)
 		)
-		(property "LCSC Part #" ""
+		(property "LCSC Part #" "C15525"
 			(at 45.72 93.98 0)
 			(hide yes)
@@
 			)
 		)
-		(property "Part #" ""
+		(property "Part #" "CL05A106MQ5NUNC"
 			(at 45.72 93.98 0)
 			(hide yes)
@@
 			)
 		)
-		(property "LCSC Part #" ""
+		(property "LCSC Part #" "C15525"
 			(at 124.46 52.07 0)
 			(hide yes)
@@
 			)
 		)
-		(property "Part #" ""
+		(property "Part #" "CL05A106MQ5NUNC"
 			(at 124.46 52.07 0)
 			(hide yes)
@@
 			)
 		)
-		(property "LCSC Part #" ""
+		(property "LCSC Part #" "C307331"
 			(at 58.42 93.98 0)
 			(hide yes)
@@
 			)
 		)
-		(property "Part #" ""
+		(property "Part #" "CL05B104KB54PNC"
 			(at 58.42 93.98 0)
 			(hide yes)
@@
 			)
 		)
-		(property "LCSC Part #" ""
+		(property "LCSC Part #" "C307331"
 			(at 58.42 86.36 0)
 			(hide yes)
@@
 			)
 		)
-		(property "Part #" ""
+		(property "Part #" "CL05B104KB54PNC"
 			(at 58.42 86.36 0)
 			(hide yes)
@@
 			)
 		)
-		(property "LCSC Part #" ""
+		(property "LCSC Part #" "C307331"
 			(at 111.76 85.09 0)
 			(hide yes)
@@
 			)
 		)
-		(property "Part #" ""
+		(property "Part #" "CL05B104KB54PNC"
 			(at 111.76 85.09 0)
 			(hide yes)
@@
 			)
 		)
-		(property "LCSC Part #" ""
+		(property "LCSC Part #" "C307331"
 			(at 111.76 52.07 0)
 			(hide yes)
@@
 			)
 		)
-		(property "Part #" ""
+		(property "Part #" "CL05B104KB54PNC"
 			(at 111.76 52.07 0)
 			(hide yes)
