File: power.kicad_sch (KiCad schematic)
At the start: 15 parts, among them J1 GT-USB-7010ASV, P1 S2B-PH-SM4-TB, U1 BQ25185DLHR, U2 TPS73633DBVT

Commit message: finish power schematic
Parts:
- added C4: 22µF, Package_DFN_QFN:VQFN-16-1EP_3x3mm_P0.5mm_EP1.6x1.6mm, symbol Device:C
- added C5: 47µF, Package_DFN_QFN:VQFN-16-1EP_3x3mm_P0.5mm_EP1.6x1.6mm, symbol Device:C
- added C6: 10nF, symbol Device:C_Small
- added C7, C8: 1µF low ESR, symbol Device:C_Small
- added L1: 1μH, symbol Device:L_Small
- added R10: 100K?, symbol Device:R_Small
- added R8: 91K, symbol Device:R_Small
- added R9: 511K, symbol Device:R_Small
- added U3: TPS631000DRLR, TPS631000DRLR:SOT50P160X60-8N, symbol TPS631000DRLR:TPS631000DRLR
Connections:
- net +3V3: now also C5.2, R9.2, U3.1 (VOUT)
- net GND: now also U2.2 (GND), C4.1, C5.1, C6.1, C7.1, C8.1, R10.2, R8.1, U3.6 (MODE), U3.7 (GND)
- net VSYS: now also U2.1 (IN), C4.2, C7.2, U3.4 (VIN), U3.5 (EN)
- net IO_AUDIO_EN: now reaches U2.3 (EN)
- net IO_AUDIO_EN: now also R10.1
- net at U2.4 (NR/FB): now also C6.2
- net 3V3_AUDIO: now reaches U2.5 (OUT)
- net 3V3_AUDIO: now also C8.2
- net CHG_STAT1 renamed IO_CHG_STAT1
- net CHG_STAT2 renamed IO_CHG_STAT2
- net VBAT: no longer names the net of C3.2, P1.1, U1.2 (BAT)
- new net: L1.1, U3.3 (LX1)
- new net: L1.2, U3.2 (LX2)
- new net: R8.2, R9.1, U3.8 (FB)
Other:
- note added: "Charge always enabled"
- note added: "Low = low-power mode"
- moved on the sheet: C1, C2, C3, P1, R1, R4, R5, R6, R7

Commit message: mcu & audio
Parts:
- added C9: 100nF, symbol Device:C
- added R11: 570K?, symbol Device:R
- added R12: 330K?, symbol Device:R
- C7, C8: value 1µF low ESR -> 1µF
- R1: value 5K -> 5K?
- R10: value 100K? -> 10K?
Connections:
- net GND: now also C9.2, R12.2
- net VBAT: now reaches C3.2, P1.1, U1.2 (BAT)
- net VBAT: now also R11.1
- net 3V3_AUDIO renamed +3V3_AUDIO
- net USB_DM renamed USB_D-
- net USB_DP renamed USB_D+
- new net IO_BAT_V: C9.1, R11.2, R12.1
- no-connect marks 0 -> 2
Other:
- note added: "Battery Voltage Monitor"
- moved on the sheet: J1, P1

Commit message: add usb data esd
Parts:
- added U8: USBLC6-2SC6, Package_TO_SOT_SMD:SOT-23-6, symbol Power_Protection:USBLC6-2SC6
- R1: value 5K? -> 18K
- R10: value 10K? -> 10K
- R11: value 570K? -> 570K
- R12: value 330K? -> 330K
Connections:
- net GND: now also U8.2 (GND)
- net USB_D+: now also U8.6 (I/O1); no longer J1.A6 (D+_A), J1.B6 (D+_B)
- net USB_D-: now also U8.4 (I/O2); no longer J1.A7 (D-_A), J1.B7 (D-_B)
- net VBUS: now also U8.5 (VBUS)
- new net: J1.A6 (D+_A), J1.B6 (D+_B), U8.1 (I/O1)
- new net: J1.A7 (D-_A), J1.B7 (D-_B), U8.3 (I/O2)

Commit message: work on pcb
Parts:
- P1: footprint S2B-PH-SM4-TB:JST_S2B-PH-SM4-TB -> battery-connector:JST_S2B-PH-SM4-TB
- U2: footprint TPS73633DBVT:SOT95P280X145-5N -> ldo:SOT95P280X145-5N
- U3: footprint TPS631000DRLR:SOT50P160X60-8N -> buck-boost:SOT50P160X60-8N
Changed lines of the file:
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@@
 			)
 		)
-		(property "Footprint" "TPS73633DBVT:SOT95P280X145-5N"
+		(property "Footprint" "ldo:SOT95P280X145-5N"
 			(at 62.23 129.54 0)
 			(hide yes)
@@
 			)
 		)
-		(property "Footprint" "S2B-PH-SM4-TB:JST_S2B-PH-SM4-TB"
+		(property "Footprint" "battery-connector:JST_S2B-PH-SM4-TB"
 			(at 256.54 44.45 0)
 			(hide yes)
@@
 			)
 		)
-		(property "Footprint" "TPS631000DRLR:SOT50P160X60-8N"
+		(property "Footprint" "buck-boost:SOT50P160X60-8N"
 			(at 209.55 125.73 0)
 			(hide yes)

Commit message: fucker
Parts:
- removed U8: USBLC6-2SC6, Package_TO_SOT_SMD:SOT-23-6, symbol Power_Protection:USBLC6-2SC6
- P1: footprint battery-connector:JST_S2B-PH-SM4-TB -> S2B-PH-SM4-TB:JST_S2B-PH-SM4-TB
- R1: value 18K -> 5K?
- R10: value 10K -> 10K?
- R11: value 570K -> 570K?
- R12: value 330K -> 330K?
- U2: footprint ldo:SOT95P280X145-5N -> TPS73633DBVT:SOT95P280X145-5N
- U3: footprint buck-boost:SOT50P160X60-8N -> TPS631000DRLR:SOT50P160X60-8N
Connections:
- net USB_D+: now also J1.A6 (D+_A), J1.B6 (D+_B)
- net USB_D-: now also J1.A7 (D-_A), J1.B7 (D-_B)

Commit message: Finish? schematic
Parts:
- removed R6: 10K, symbol Device:R_Small
- added NT1: NetTie_2, symbol Device:NetTie_2
- added R21: 10K, symbol Device:R_Small
- added U5: USBLC6-2SC6, Package_TO_SOT_SMD:SOT-23-6, symbol Power_Protection:USBLC6-2SC6
- P1: footprint S2B-PH-SM4-TB:JST_S2B-PH-SM4-TB -> battery-connector:JST_S2B-PH-SM4-TB
- R1: value 5K? -> 18K
- U2: footprint TPS73633DBVT:SOT95P280X145-5N -> ldo:SOT95P280X145-5N
- U3: footprint TPS631000DRLR:SOT50P160X60-8N -> buck-boost:SOT50P160X60-8N
Connections:
- net +3V3: now also R21.2
- net GND: now also D1.2 (A2), NT1.1, U5.2 (GND); no longer D1.1 (A1), U2.2 (GND)
- net IO_CHG_STAT1: now also R21.1
- net USB_D+: now also U5.6 (I/O1); no longer J1.A6 (D+_A), J1.B6 (D+_B)
- net USB_D-: now also U5.4 (I/O2); no longer J1.A7 (D-_A), J1.B7 (D-_B)
- net VBUS: now also D1.1 (A1), U5.5 (VBUS); no longer D1.2 (A2)
- new net: J1.A6 (D+_A), J1.B6 (D+_B), U5.1 (I/O1)
- new net: J1.A7 (D-_A), J1.B7 (D-_B), U5.3 (I/O2)
- new net GNDA: NT1.2, U2.2 (GND)

Commit message: holy routing
Parts:
- C1, C2, C3, C4, C5: footprint Package_DFN_QFN:VQFN-16-1EP_3x3mm_P0.5mm_EP1.6x1.6mm -> Capacitor_SMD:C_0201_0603Metric
- C6, C7, C8, C9: footprint (none) -> Capacitor_SMD:C_0201_0603Metric
- L1: footprint (none) -> Inductor_SMD:L_0201_0603Metric
- NT1: footprint (none) -> NetTie:NetTie-2_SMD_Pad0.5mm
- R1, R10, R11, R12, R2, R21, R3, R4, R5, R7, R8, R9: footprint (none) -> Resistor_SMD:R_0201_0603Metric
Connections:
- net GND: no longer C6.1, C8.1
- net GNDA: now also C6.1, C8.1
- net USB_D+: now also J1.A6 (D+_A), J1.B6 (D+_B), U5.3 (I/O2), U5.4 (I/O2); no longer U5.6 (I/O1)
- net USB_D-: now also J1.A7 (D-_A), J1.B7 (D-_B), U5.1 (I/O1), U5.6 (I/O1); no longer U5.4 (I/O2)
Other:
- moved on the sheet: U5

Commit message: fix sd card pullups
Other:
- moved on the sheet: C9, R11, R12
Changed lines of the file:
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@@
 	)
 	(junction
-		(at 247.65 77.47)
+		(at 247.65 81.28)
 		(diameter 0)
 		(color 0 0 0 0)
@@
 	)
 	(junction
-		(at 259.08 77.47)
+		(at 259.08 81.28)
 		(diameter 0)
 		(color 0 0 0 0)
@@
 	(wire
 		(pts
-			(xy 259.08 77.47) (xy 262.89 77.47)
+			(xy 259.08 81.28) (xy 262.89 81.28)
 		)
 		(stroke
@@
 	(wire
 		(pts
-			(xy 247.65 66.04) (xy 247.65 68.58)
+			(xy 247.65 69.85) (xy 247.65 72.39)
 		)
 		(stroke
@@
 	(wire
 		(pts
-			(xy 247.65 76.2) (xy 247.65 77.47)
+			(xy 247.65 80.01) (xy 247.65 81.28)
 		)
 		(stroke
@@
 	(wire
 		(pts
-			(xy 247.65 77.47) (xy 259.08 77.47)
+			(xy 247.65 81.28) (xy 259.08 81.28)
 		)
 		(stroke
@@
 	(wire
 		(pts
-			(xy 247.65 77.47) (xy 247.65 80.01)
+			(xy 247.65 81.28) (xy 247.65 83.82)
 		)
 		(stroke
@@
 	(wire
 		(pts
-			(xy 259.08 80.01) (xy 259.08 77.47)
+			(xy 259.08 83.82) (xy 259.08 81.28)
 		)
 		(stroke
@@
 		)
 	)
-	(label "USB_D+"
-		(at 74.93 53.34 0)
+	(label "VBAT"
+		(at 227.33 40.64 0)
 		(effects
 			(font
@@
 		)
 	)
-	(label "VBAT"
-		(at 227.33 40.64 0)
+	(label "USB_D+"
+		(at 74.93 53.34 0)
 		(effects
 			(font
@@
 	)
 	(label "VBAT"
-		(at 247.65 66.04 0)
+		(at 251.46 43.18 180)
 		(effects
 			(font
 				(size 1.27 1.27)
 			)
-			(justify left bottom)
+			(justify right bottom)
 		)
 	)
@@
 		)
 	)
-	(label "VBAT"
-		(at 251.46 43.18 180)
+	(label "USB_D-"
+		(at 39.37 55.88 180)
 		(effects
 			(font
@@
 		)
 	)
-	(label "USB_D-"
-		(at 39.37 55.88 180)
+	(label "VBAT"
+		(at 247.65 69.85 0)
 		(effects
 			(font
 				(size 1.27 1.27)
 			)
-			(justify right bottom)
+			(justify left bottom)
 		)
 	)
@@
 	(hierarchical_label "IO_BAT_V"
 		(shape input)
-		(at 262.89 77.47 0)
+		(at 262.89 81.28 0)
 		(effects
 			(font
@@
 	(symbol
 		(lib_id "power:GND")
-		(at 259.08 87.63 0)
+		(at 259.08 91.44 0)
 		(unit 1)
 		(body_style 1)
@@
 		(fields_autoplaced yes)
 		(property "Reference" "#PWR029"
-			(at 259.08 93.98 0)
+			(at 259.08 97.79 0)
 			(hide yes)
 			(show_name no)
@@
 		)
 		(property "Value" "GND"
-			(at 259.08 92.71 0)
+			(at 259.08 96.52 0)
 			(show_name no)
 			(do_not_autoplace no)
@@
 		)
 		(property "Footprint" ""
-			(at 259.08 87.63 0)
+			(at 259.08 91.44 0)
 			(hide yes)
 			(show_name no)
@@
 		)
 		(property "Datasheet" ""
-			(at 259.08 87.63 0)
+			(at 259.08 91.44 0)
 			(hide yes)
 			(show_name no)
@@
 		)
 		(property "Description" "Power symbol creates a global label with name \"GND\" , ground"
-			(at 259.08 87.63 0)
+			(at 259.08 91.44 0)
 			(hide yes)
 			(show_name no)
@@
 	(symbol
 		(lib_id "Device:R")
-		(at 247.65 72.39 0)
+		(at 247.65 76.2 0)
 		(unit 1)
 		(body_style 1)
@@
 		(fields_autoplaced yes)
 		(property "Reference" "R11"
-			(at 250.19 71.1199 0)
+			(at 250.19 74.9299 0)
 			(show_name no)
 			(do_not_autoplace no)
@@
 		)
 		(property "Value" "570K?"
-			(at 250.19 73.6599 0)
+			(at 250.19 77.4699 0)
 			(show_name no)
 			(do_not_autoplace no)
@@
 		)
 		(property "Footprint" "Resistor_SMD:R_0201_0603Metric"
-			(at 245.872 72.39 90)
+			(at 245.872 76.2 90)
 			(hide yes)
 			(show_name no)
@@
 		)
 		(property "Datasheet" ""
-			(at 247.65 72.39 0)
+			(at 247.65 76.2 0)
 			(hide yes)
 			(show_name no)
@@
 		)
 		(property "Description" "Resistor"
-			(at 247.65 72.39 0)
+			(at 247.65 76.2 0)
 			(hide yes)
 			(show_name no)
@@
 	(symbol
 		(lib_id "Device:R")
-		(at 247.65 83.82 0)
+		(at 247.65 87.63 0)
 		(unit 1)
 		(body_style 1)
@@
 		(fields_autoplaced yes)
 		(property "Reference" "R12"
-			(at 250.19 82.5499 0)
+			(at 250.19 86.3599 0)
 			(show_name no)
 			(do_not_autoplace no)
@@
 		)
 		(property "Value" "330K?"
-			(at 250.19 85.0899 0)
+			(at 250.19 88.8999 0)
 			(show_name no)
 			(do_not_autoplace no)
@@
 		)
 		(property "Footprint" "Resistor_SMD:R_0201_0603Metric"
-			(at 245.872 83.82 90)
+			(at 245.872 87.63 90)
 			(hide yes)
 			(show_name no)
@@
 		)
 		(property "Datasheet" ""
-			(at 247.65 83.82 0)
+			(at 247.65 87.63 0)
 			(hide yes)
 			(show_name no)
@@
 		)
 		(property "Description" "Resistor"
-			(at 247.65 83.82 0)
+			(at 247.65 87.63 0)
 			(hide yes)
 			(show_name no)
@@
 	(symbol
 		(lib_id "Device:C")
-		(at 259.08 83.82 0)
+		(at 259.08 87.63 0)
 		(unit 1)
 		(body_style 1)
@@
 		(fields_autoplaced yes)
 		(property "Reference" "C9"
-			(at 262.89 82.5499 0)
+			(at 262.89 86.3599 0)
 			(show_name no)
 			(do_not_autoplace no)
@@
 		)
 		(property "Value" "100nF"
-			(at 262.89 85.0899 0)
+			(at 262.89 88.8999 0)
 			(show_name no)
 			(do_not_autoplace no)
@@
 		)
 		(property "Footprint" "Capacitor_SMD:C_0201_0603Metric"
-			(at 260.0452 87.63 0)
+			(at 260.0452 91.44 0)
 			(hide yes)
 			(show_name no)
@@
 		)
 		(property "Datasheet" ""
-			(at 259.08 83.82 0)
+			(at 259.08 87.63 0)
 			(hide yes)
 			(show_name no)
@@
 		)
 		(property "Description" "Unpolarized capacitor"
-			(at 259.08 83.82 0)
+			(at 259.08 87.63 0)
 			(hide yes)
 			(show_name no)
@@
 	(symbol
 		(lib_id "power:GND")
-		(at 247.65 87.63 0)
+		(at 247.65 91.44 0)
 		(unit 1)
 		(body_style 1)
@@
 		(fields_autoplaced yes)
 		(property "Reference" "#PWR028"
-			(at 247.65 93.98 0)
+			(at 247.65 97.79 0)
 			(hide yes)
 			(show_name no)
@@
 		)
 		(property "Value" "GND"
-			(at 247.65 92.71 0)
+			(at 247.65 96.52 0)
 			(show_name no)
 			(do_not_autoplace no)
@@
 		)
 		(property "Footprint" ""
-			(at 247.65 87.63 0)
+			(at 247.65 91.44 0)
 			(hide yes)
 			(show_name no)
@@
 		)
 		(property "Datasheet" ""
-			(at 247.65 87.63 0)
+			(at 247.65 91.44 0)
 			(hide yes)
 			(show_name no)
@@
 		)
 		(property "Description" "Power symbol creates a global label with name \"GND\" , ground"
-			(at 247.65 87.63 0)
+			(at 247.65 91.44 0)
 			(hide yes)
 			(show_name no)
