File: power.kicad_sch (KiCad schematic)
At the start: 30 parts, among them J1 GT-USB-7010ASV, P1 S2B-PH-SM4-TB, U1 BQ25185DLHR, U2 TPS73633DBVT, U3 TPS631000DRLR, U5 USBLC6-2SC6

Commit message: switch to stm32, wire audio section
Parts:
- C1, C2, C3, C4, C5, C6, C7, C8, C9: footprint Capacitor_SMD:C_0201_0603Metric -> Capacitor_SMD:C_0402_1005Metric
- L1: footprint Inductor_SMD:L_0201_0603Metric -> Inductor_SMD:L_1008_2520Metric
- R1, R10, R11, R12, R2, R21, R3, R4, R5, R7, R8, R9: footprint Resistor_SMD:R_0201_0603Metric -> Resistor_SMD:R_0402_1005Metric
Connections:
- net GND: now also U2.2 (GND)
- net GNDA: no longer U2.2 (GND)
Changed lines of the file:
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@@
 			)
 		)
-		(property "Footprint" "Resistor_SMD:R_0201_0603Metric"
+		(property "Footprint" "Resistor_SMD:R_0402_1005Metric"
 			(at 156.21 45.72 0)
 			(hide yes)
@@
 			)
 		)
-		(property "Footprint" "Capacitor_SMD:C_0201_0603Metric"
+		(property "Footprint" "Capacitor_SMD:C_0402_1005Metric"
 			(at 96.52 119.38 0)
 			(hide yes)
@@
 			)
 		)
-		(property "Footprint" "Resistor_SMD:R_0201_0603Metric"
+		(property "Footprint" "Resistor_SMD:R_0402_1005Metric"
 			(at 245.872 76.2 90)
 			(hide yes)
@@
 			)
 		)
-		(property "Footprint" "Resistor_SMD:R_0201_0603Metric"
+		(property "Footprint" "Resistor_SMD:R_0402_1005Metric"
 			(at 86.36 60.96 0)
 			(hide yes)
@@
 			)
 		)
-		(property "Footprint" "Resistor_SMD:R_0201_0603Metric"
+		(property "Footprint" "Resistor_SMD:R_0402_1005Metric"
 			(at 245.872 87.63 90)
 			(hide yes)
@@
 			)
 		)
-		(property "Footprint" "Capacitor_SMD:C_0201_0603Metric"
+		(property "Footprint" "Capacitor_SMD:C_0402_1005Metric"
 			(at 260.0452 91.44 0)
 			(hide yes)
@@
 			)
 		)
-		(property "Footprint" "Capacitor_SMD:C_0201_0603Metric"
+		(property "Footprint" "Capacitor_SMD:C_0402_1005Metric"
 			(at 247.9548 115.57 0)
 			(hide yes)
@@
 			)
 		)
-		(property "Footprint" "Capacitor_SMD:C_0201_0603Metric"
+		(property "Footprint" "Capacitor_SMD:C_0402_1005Metric"
 			(at 191.4652 115.57 0)
 			(hide yes)
@@
 			)
 		)
-		(property "Footprint" "Capacitor_SMD:C_0201_0603Metric"
+		(property "Footprint" "Capacitor_SMD:C_0402_1005Metric"
 			(at 41.91 129.54 0)
 			(hide yes)
@@
 			)
 		)
-		(property "Footprint" "Inductor_SMD:L_0201_0603Metric"
+		(property "Footprint" "Inductor_SMD:L_1008_2520Metric"
 			(at 227.33 121.92 0)
 			(hide yes)
@@
 			)
 		)
-		(property "Footprint" "Capacitor_SMD:C_0201_0603Metric"
+		(property "Footprint" "Capacitor_SMD:C_0402_1005Metric"
 			(at 167.9448 26.67 0)
 			(hide yes)
@@
 			)
 		)
-		(property "Footprint" "Resistor_SMD:R_0201_0603Metric"
+		(property "Footprint" "Resistor_SMD:R_0402_1005Metric"
 			(at 237.49 123.19 0)
 			(hide yes)
@@
 			)
 		)
-		(property "Footprint" "Resistor_SMD:R_0201_0603Metric"
+		(property "Footprint" "Resistor_SMD:R_0402_1005Metric"
 			(at 49.53 111.76 0)
 			(hide yes)
@@
 			)
 		)
-		(property "Footprint" "Capacitor_SMD:C_0201_0603Metric"
+		(property "Footprint" "Capacitor_SMD:C_0402_1005Metric"
 			(at 222.5548 40.64 0)
 			(hide yes)
@@
 			)
 		)
-		(property "Footprint" "Resistor_SMD:R_0201_0603Metric"
+		(property "Footprint" "Resistor_SMD:R_0402_1005Metric"
 			(at 163.83 58.42 0)
 			(hide yes)
@@
 			)
 		)
-		(property "Footprint" "Resistor_SMD:R_0201_0603Metric"
+		(property "Footprint" "Resistor_SMD:R_0402_1005Metric"
 			(at 167.64 58.42 0)
 			(hide yes)
@@
 			)
 		)
-		(property "Footprint" "Resistor_SMD:R_0201_0603Metric"
+		(property "Footprint" "Resistor_SMD:R_0402_1005Metric"
 			(at 209.55 45.72 0)
 			(hide yes)
@@
 			)
 		)
-		(property "Value" "GNDA"
+		(property "Value" "GND"
 			(at 83.82 134.6199 90)
 			(show_name no)
@@
 			)
 		)
-		(property "Footprint" "Resistor_SMD:R_0201_0603Metric"
+		(property "Footprint" "Resistor_SMD:R_0402_1005Metric"
 			(at 237.49 135.89 0)
 			(hide yes)
@@
 			)
 		)
-		(property "Footprint" "Capacitor_SMD:C_0201_0603Metric"
+		(property "Footprint" "Capacitor_SMD:C_0402_1005Metric"
 			(at 30.48 121.92 0)
 			(hide yes)
@@
 			)
 		)
-		(property "Footprint" "Resistor_SMD:R_0201_0603Metric"
+		(property "Footprint" "Resistor_SMD:R_0402_1005Metric"
 			(at 156.21 38.1 0)
 			(hide yes)
@@
 			)
 		)
-		(property "Footprint" "Capacitor_SMD:C_0201_0603Metric"
+		(property "Footprint" "Capacitor_SMD:C_0402_1005Metric"
 			(at 215.5952 27.94 0)
 			(hide yes)
@@
 			)
 		)
-		(property "Footprint" "Resistor_SMD:R_0201_0603Metric"
+		(property "Footprint" "Resistor_SMD:R_0402_1005Metric"
 			(at 29.21 50.8 0)
 			(hide yes)

Commit message: some fixes
Connections:
- net USB_D+: no longer J1.A6 (D+_A), J1.B6 (D+_B), U5.3 (I/O2)
- net USB_D-: no longer J1.A7 (D-_A), J1.B7 (D-_B), U5.1 (I/O1)
- new net USB_DN: J1.A7 (D-_A), J1.B7 (D-_B), U5.1 (I/O1)
- new net USB_DP: J1.A6 (D+_A), J1.B6 (D+_B), U5.3 (I/O2)
Changed lines of the file:
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@@
+		)
+	)
+	(label "USB_DP"
+		(at 39.37 53.34 180)
+		(effects
+			(font
+				(size 1.27 1.27)
+			)
+			(justify right bottom)
 		)
 	)
@@
 		)
 	)
-	(label "USB_D+"
+	(label "USB_DP"
 		(at 74.93 53.34 0)
 		(effects
@@
 		)
 	)
-	(label "USB_D-"
+	(label "USB_DN"
 		(at 74.93 55.88 0)
 		(effects
@@
 			)
 			(justify left bottom)
-		)
-	)
-	(label "USB_D-"
-		(at 39.37 55.88 180)
-		(effects
-			(font
-				(size 1.27 1.27)
-			)
-			(justify right bottom)
 		)
 	)
@@
 		)
 	)
-	(label "USB_D+"
-		(at 39.37 53.34 180)
+	(label "USB_DN"
+		(at 39.37 55.88 180)
 		(effects
 			(font

Commit message: add mpns to buck boost
Parts:
- C4: footprint Capacitor_SMD:C_0402_1005Metric -> Capacitor_SMD:C_0603_1608Metric; LCSC Part # (none) -> C59461; Part # (none) -> CL10A226MQ8NRNC
- C5: footprint Capacitor_SMD:C_0402_1005Metric -> Capacitor_SMD:C_0805_2012Metric; LCSC Part # (none) -> C16780; Part # (none) -> CL21A476MQYNNNE
- L1: LCSC Part # (none) -> C882955; Part # (none) -> DFE252012P-1R0M=P2
- R8: footprint Resistor_SMD:R_0402_1005Metric -> Resistor_SMD:R_0603_1608Metric; LCSC Part # (none) -> C23265; Part # (none) -> 0603WAF9102T5E
- R9: value 511K -> 510K; footprint Resistor_SMD:R_0402_1005Metric -> Resistor_SMD:R_0603_1608Metric; LCSC Part # (none) -> C23192; Part # (none) -> 0603WAF5103T5E
- U3: LCSC Part # (none) -> C5219190; Part # (none) -> TPS631000DRLR

Commit message: fill more parts
Parts:
- P1: LCSC Part # (none) -> C54582899; Part # (none) -> XY-S2B-PH-SM4-TB
- R2, R3: LCSC Part # (none) -> C25905; Part # (none) -> 0402WGF5101TCE
- U5: LCSC Part # (none) -> C7519; Part # (none) -> ST USBLC6-2SC6
Changed lines of the file:
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@@
 			)
 		)
-		(property "LCSC Part #" ""
+		(property "LCSC Part #" "C7519"
 			(at 102.87 55.88 0)
 			(hide yes)
@@
 			)
 		)
-		(property "Part #" ""
+		(property "Part #" "ST USBLC6-2SC6"
 			(at 102.87 55.88 0)
 			(hide yes)
@@
 			)
 		)
-		(property "LCSC Part #" ""
+		(property "LCSC Part #" "C25905"
 			(at 86.36 60.96 0)
 			(hide yes)
@@
 			)
 		)
-		(property "Part #" ""
+		(property "Part #" "0402WGF5101TCE"
 			(at 86.36 60.96 0)
 			(hide yes)
@@
 			)
 		)
-		(property "LCSC Part #" ""
+		(property "LCSC Part #" "C54582899"
 			(at 256.54 44.45 0)
 			(hide yes)
@@
 			)
 		)
-		(property "Part #" ""
+		(property "Part #" "XY-S2B-PH-SM4-TB"
 			(at 256.54 44.45 0)
 			(hide yes)
@@
 			)
 		)
-		(property "LCSC Part #" ""
+		(property "LCSC Part #" "C25905"
 			(at 29.21 50.8 90)
 			(hide yes)
@@
 			)
 		)
-		(property "Part #" ""
+		(property "Part #" "0402WGF5101TCE"
 			(at 29.21 50.8 90)
 			(hide yes)

Commit message: Finish all power MPNs
Parts:
- C1, C3: footprint Capacitor_SMD:C_0402_1005Metric -> Capacitor_SMD:C_0603_1608Metric; LCSC Part # (none) -> C15849; Part # (none) -> CL10A105KB8NNNC
- C2: footprint Capacitor_SMD:C_0402_1005Metric -> Capacitor_SMD:C_0603_1608Metric; LCSC Part # (none) -> C96446; Part # (none) -> CL10A106MA8NRNC
- C6: LCSC Part # (none) -> C15195; Part # (none) -> CL05B103KB5NNNC
- C7, C8: LCSC Part # (none) -> C52923; Part # (none) -> CL05A105KA5NQNC
- C9: LCSC Part # (none) -> C1525; Part # (none) -> CL05B104KO5NNNC
- J1: LCSC Part # (none) -> C2988369; Part # (none) -> GT-USB-7010ASV
- R1: LCSC Part # (none) -> C25762; Part # (none) -> 0402WGF1802TCE
- R11: value 570K? -> 470K; LCSC Part # (none) -> C25790; Part # (none) -> 0402WGF4703TCE
- R12: value 330K? -> 470K; LCSC Part # (none) -> C25790; Part # (none) -> 0402WGF4703TCE
- R21, R5, R7: LCSC Part # (none) -> C25744; Part # (none) -> 0402WGF1002TCE
- R4: LCSC Part # (none) -> C11702; Part # (none) -> 0402WGF1001TCE
- U1: LCSC Part # (none) -> C19725033; Part # (none) -> BQ25185DLHR
- U2: LCSC Part # (none) -> C2864221; Part # (none) -> TPS73633DBVT
Changed lines of the file:
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@@
 			)
 		)
-		(property "LCSC Part #" ""
+		(property "LCSC Part #" "C25744"
 			(at 156.21 45.72 0)
 			(hide yes)
@@
 			)
 		)
-		(property "Part #" ""
+		(property "Part #" "0402WGF1002TCE"
 			(at 156.21 45.72 0)
 			(hide yes)
@@
 			)
 		)
-		(property "LCSC Part #" ""
+		(property "LCSC Part #" "C52923"
 			(at 96.52 119.38 0)
 			(hide yes)
@@
 			)
 		)
-		(property "Part #" ""
+		(property "Part #" "CL05A105KA5NQNC"
 			(at 96.52 119.38 0)
 			(hide yes)
@@
 			)
 		)
-		(property "Value" "570K?"
+		(property "Value" "470K"
 			(at 250.19 77.4699 0)
 			(show_name no)
@@
 			)
 		)
-		(property "LCSC Part #" ""
+		(property "LCSC Part #" "C25790"
 			(at 247.65 76.2 0)
 			(hide yes)
@@
 			)
 		)
-		(property "Part #" ""
+		(property "Part #" "0402WGF4703TCE"
 			(at 247.65 76.2 0)
 			(hide yes)
@@
 			)
 		)
-		(property "LCSC Part #" ""
+		(property "LCSC Part #" "C19725033"
 			(at 189.23 48.26 0)
 			(hide yes)
@@
 			)
 		)
-		(property "Part #" ""
+		(property "Part #" "BQ25185DLHR"
 			(at 189.23 48.26 0)
 			(hide yes)
@@
 			)
 		)
-		(property "Value" "330K?"
+		(property "Value" "470K"
 			(at 250.19 88.8999 0)
 			(show_name no)
@@
 			)
 		)
-		(property "LCSC Part #" ""
+		(property "LCSC Part #" "C25790"
 			(at 247.65 87.63 0)
 			(hide yes)
@@
 			)
 		)
-		(property "Part #" ""
+		(property "Part #" "0402WGF4703TCE"
 			(at 247.65 87.63 0)
 			(hide yes)
@@
 			)
 		)
-		(property "LCSC Part #" ""
+		(property "LCSC Part #" "C2864221"
 			(at 62.23 129.54 0)
 			(hide yes)
@@
 			)
 		)
-		(property "Part #" ""
+		(property "Part #" "TPS73633DBVT"
 			(at 62.23 129.54 0)
 			(hide yes)
@@
 			)
 		)
-		(property "LCSC Part #" ""
+		(property "LCSC Part #" "C1525"
 			(at 259.08 87.63 0)
 			(hide yes)
@@
 			)
 		)
-		(property "Part #" ""
+		(property "Part #" "CL05B104KO5NNNC"
 			(at 259.08 87.63 0)
 			(hide yes)
@@
 			)
 		)
-		(property "LCSC Part #" ""
+		(property "LCSC Part #" "C15195"
 			(at 41.91 129.54 90)
 			(hide yes)
@@
 			)
 		)
-		(property "Part #" ""
+		(property "Part #" "CL05B103KB5NNNC"
 			(at 41.91 129.54 90)
 			(hide yes)
@@
 			)
 		)
-		(property "Footprint" "Capacitor_SMD:C_0402_1005Metric"
+		(property "Footprint" "Capacitor_SMD:C_0603_1608Metric"
 			(at 167.9448 26.67 0)
 			(hide yes)
@@
 			)
 		)
-		(property "LCSC Part #" ""
+		(property "LCSC Part #" "C15849"
 			(at 168.91 30.48 0)
 			(hide yes)
@@
 			)
 		)
-		(property "Part #" ""
+		(property "Part #" "CL10A105KB8NNNC"
 			(at 168.91 30.48 0)
 			(hide yes)
@@
 			)
 		)
-		(property "Footprint" "Capacitor_SMD:C_0402_1005Metric"
+		(property "Footprint" "Capacitor_SMD:C_0603_1608Metric"
 			(at 222.5548 40.64 0)
 			(hide yes)
@@
 			)
 		)
-		(property "LCSC Part #" ""
+		(property "LCSC Part #" "C15849"
 			(at 223.52 44.45 0)
 			(hide yes)
@@
 			)
 		)
-		(property "Part #" ""
+		(property "Part #" "CL10A105KB8NNNC"
 			(at 223.52 44.45 0)
 			(hide yes)
@@
 			)
 		)
-		(property "LCSC Part #" ""
+		(property "LCSC Part #" "C25762"
 			(at 163.83 58.42 0)
 			(hide yes)
@@
 			)
 		)
-		(property "Part #" ""
+		(property "Part #" "0402WGF1802TCE"
 			(at 163.83 58.42 0)
 			(hide yes)
@@
 			)
 		)
-		(property "LCSC Part #" ""
+		(property "LCSC Part #" "C11702"
 			(at 167.64 58.42 0)
 			(hide yes)
@@
 			)
 		)
-		(property "Part #" ""
+		(property "Part #" "0402WGF1001TCE"
 			(at 167.64 58.42 0)
 			(hide yes)
@@
 			)
 		)
-		(property "LCSC Part #" ""
+		(property "LCSC Part #" "C25744"
 			(at 209.55 45.72 90)
 			(hide yes)
@@
 			)
 		)
-		(property "Part #" ""
+		(property "Part #" "0402WGF1002TCE"
 			(at 209.55 45.72 90)
 			(hide yes)
@@
 			)
 		)
-		(property "LCSC Part #" ""
+		(property "LCSC Part #" "C2988369"
 			(at 57.15 55.88 0)
 			(hide yes)
@@
 			)
 		)
-		(property "Part #" ""
+		(property "Part #" "GT-USB-7010ASV"
 			(at 57.15 55.88 0)
 			(hide yes)
@@
 			)
 		)
-		(property "LCSC Part #" ""
+		(property "LCSC Part #" "C52923"
 			(at 30.48 121.92 0)
 			(hide yes)
@@
 			)
 		)
-		(property "Part #" ""
+		(property "Part #" "CL05A105KA5NQNC"
 			(at 30.48 121.92 0)
 			(hide yes)
@@
 			)
 		)
-		(property "LCSC Part #" ""
+		(property "LCSC Part #" "C25744"
 			(at 156.21 38.1 0)
 			(hide yes)
@@
 			)
 		)
-		(property "Part #" ""
+		(property "Part #" "0402WGF1002TCE"
 			(at 156.21 38.1 0)
 			(hide yes)
@@
 			)
 		)
-		(property "Footprint" "Capacitor_SMD:C_0402_1005Metric"
+		(property "Footprint" "Capacitor_SMD:C_0603_1608Metric"
 			(at 215.5952 27.94 0)
 			(hide yes)
@@
 			)
 		)
-		(property "LCSC Part #" ""
+		(property "LCSC Part #" "C96446"
 			(at 214.63 31.75 0)
 			(hide yes)
@@
 			)
 		)
-		(property "Part #" ""
+		(property "Part #" "CL10A106MA8NRNC"
 			(at 214.63 31.75 0)
 			(hide yes)

Commit message: label sections
Parts:
- R11: Part # 0402WGF4703TCE -> (none)
- R12: Part # 0402WGF4703TCE -> 0603WAF4703T5E
Changed lines of the file:
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@@
 			)
 		)
-		(property "Part #" "0402WGF4703TCE"
+		(property "Part #" ""
 			(at 247.65 76.2 0)
 			(hide yes)
@@
 			)
 		)
-		(property "Part #" "0402WGF4703TCE"
+		(property "Part #" "0603WAF4703T5E"
 			(at 247.65 87.63 0)
 			(hide yes)
