File: mcu.kicad_sch (KiCad schematic)
At the start: 14 parts, among them J2 DM3CS-SF, U4 ESP32-S3-WROOM-1U-N16R8, U5 ER_OLEDM0.91_1x-I2C

Commit message: work on pcb
Parts:
- removed U5: ER_OLEDM0.91_1x-I2C, Display:ER_OLEDM0.91_1x-I2C, symbol Display_Graphic:ER_OLEDM0.91_1x-I2C
- added J4: SCREEN, Connector:FanPinHeader_1x04_P2.54mm_Vertical, symbol Connector_Generic:Conn_01x04
- J2: footprint DM3CS-SF:HRS_DM3CS-SF -> microsd:HRS_DM3CS-SF
- S3, S4: footprint TL3340AF160QG:SW_TL3340AF160QG -> side-button:SW_TL3340AF160QG
- U4: footprint ESP32-S3-WROOM-1U-N16R8:XCVR_ESP32-S3-WROOM-1U-N16R8 -> esp32:XCVR_ESP32-S3-WROOM-1U-N16R8
Connections:
- net +3V3: now also J4.3 (Pin_3)
- net GND: now also J4.4 (Pin_4)
- net IO_I2C_SCL: now also J4.2 (Pin_2)
- net IO_I2C_SDA: now also J4.1 (Pin_1)
- net IO_DAC_BCK: now reaches U4.10 (IO17)
- net IO_DAC_LRCK: now reaches U4.11 (IO18)
- net IO_DAC_DIN: now reaches U4.9 (IO16)

Commit message: fucker
Parts:
- removed J4: SCREEN, Connector:FanPinHeader_1x04_P2.54mm_Vertical, symbol Connector_Generic:Conn_01x04
- added U5: ER_OLEDM0.91_1x-I2C, Display:ER_OLEDM0.91_1x-I2C, symbol Display_Graphic:ER_OLEDM0.91_1x-I2C
- J2: footprint microsd:HRS_DM3CS-SF -> DM3CS-SF:HRS_DM3CS-SF
- R14, R16, R17: value 10K? -> 10K
- S3, S4: footprint side-button:SW_TL3340AF160QG -> TL3340AF160QG:SW_TL3340AF160QG
- U4: footprint esp32:XCVR_ESP32-S3-WROOM-1U-N16R8 -> ESP32-S3-WROOM-1U-N16R8:XCVR_ESP32-S3-WROOM-1U-N16R8
Connections:
- net +3V3: now also U5.2 (VCC)
- net GND: now also U5.1 (GND)
- net IO_DAC_BCK: now also U4.29 (IO36); no longer U4.10 (IO17)
- net IO_DAC_DIN: now also U4.28 (IO35); no longer U4.9 (IO16)
- net IO_DAC_LRCK: now also U4.30 (IO37); no longer U4.11 (IO18)
- net IO_I2C_SCL: now also U5.3 (SCL)
- net IO_I2C_SDA: now also U5.4 (SDA)
- net IO_DAC_SCK: now reaches U4.23 (IO21)

Commit message: Finish? schematic
Parts:
- removed U5: ER_OLEDM0.91_1x-I2C, Display:ER_OLEDM0.91_1x-I2C, symbol Display_Graphic:ER_OLEDM0.91_1x-I2C
- added J4: SCREEN, symbol Connector_Generic:Conn_01x04
- J2: footprint DM3CS-SF:HRS_DM3CS-SF -> microsd:HRS_DM3CS-SF
- S3, S4: footprint TL3340AF160QG:SW_TL3340AF160QG -> side-button:SW_TL3340AF160QG
- U4: footprint ESP32-S3-WROOM-1U-N16R8:XCVR_ESP32-S3-WROOM-1U-N16R8 -> esp32:XCVR_ESP32-S3-WROOM-1U-N16R8
Connections:
- net +3V3: now also J4.3 (Pin_3)
- net GND: now also J4.4 (Pin_4)
- net IO_DAC_BCK: now also U4.10 (IO17); no longer U4.29 (IO36)
- net IO_DAC_DIN: now also U4.9 (IO16); no longer U4.28 (IO35)
- net IO_DAC_LRCK: now also U4.11 (IO18); no longer U4.30 (IO37)
- net IO_I2C_SCL: now also J4.2 (Pin_2)
- net IO_I2C_SDA: now also J4.1 (Pin_1)
- net IO_DAC_SCK: no longer names the net of U4.23 (IO21)
- no-connect marks 5 -> 18

Commit message: holy routing
Parts:
- added TP1: RX, TestPoint:TestPoint_Pad_1.5x1.5mm, symbol Connector:TestPoint
- added TP2: TX, TestPoint:TestPoint_Pad_1.5x1.5mm, symbol Connector:TestPoint
- added U8: SiP32431DR3, Package_TO_SOT_SMD:SOT-363_SC-70-6, symbol Power_Management:SiP32431DR3
- C10, C11: footprint (none) -> Capacitor_SMD:C_0201_0603Metric
- J4: footprint (none) -> Connector_PinHeader_2.54mm:PinHeader_1x04_P2.54mm_Vertical
- R13, R14, R15, R16, R17: footprint (none) -> Resistor_SMD:R_0201_0603Metric
Connections:
- net +3V3: now also J4.2 (Pin_2), U8.4 (IN); no longer J4.3 (Pin_3)
- net GND: now also J4.1 (Pin_1), U8.2 (GND), U8.5 (GND); no longer J4.4 (Pin_4)
- net IO_AUDIO_EN: now also U4.20 (IO12); no longer U4.8 (IO15)
- net IO_BAT_V: now also U4.19 (IO11); no longer U4.20 (IO12)
- net IO_CHG_STAT1: now also U4.18 (IO10); no longer U4.21 (IO13)
- net IO_CHG_STAT2: now also U4.17 (IO9); no longer U4.22 (IO14)
- net IO_DAC_BCK: now also U4.22 (IO14); no longer U4.10 (IO17)
- net IO_DAC_DIN: now also U4.21 (IO13); no longer U4.9 (IO16)
- net IO_I2C_SCL: now also J4.3 (Pin_3), U4.35 (IO42); no longer J4.2 (Pin_2), U4.38 (IO2)
- net IO_I2C_SDA: now also J4.4 (Pin_4), U4.34 (IO41); no longer J4.1 (Pin_1), U4.39 (IO1)
- net IO_SD_CLK: now also U4.8 (IO15); no longer U4.5 (IO5)
- net IO_SD_CMD: now also U4.7 (IO7); no longer U4.4 (IO4)
- net IO_SD_DAT0: now also U4.9 (IO16); no longer U4.6 (IO6)
- net IO_SD_DAT1: now also U4.10 (IO17); no longer U4.7 (IO7)
- net IO_SD_DAT2: now also U4.5 (IO5); no longer U4.12 (IO8)
- net IO_SD_DAT3: now also U4.6 (IO6); no longer U4.17 (IO9)
- net IO_VOLUME_DOWN: now also U4.25 (IO48); no longer U4.19 (IO11)
- net IO_VOLUME_UP: now also U4.39 (IO1); no longer U4.18 (IO10)
- net at U4.36 (RXD0): now also TP1.1
- net at U4.37 (TXD0): now also TP2.1
- net +3V3_AUDIO renamed VSD
- net VSD: now also U8.1 (OUT)
- new net IO_SD_EN: U4.4 (IO4), U8.3 (ON)
- no-connect marks 18 -> 8
Other:
- note removed: "On the audio line so we can turn the SD card on and off, because it has high idle power drain"
- moved on the sheet: R14

Commit message: some placements
Connections:
- net IO_AUDIO_EN: now also U4.21 (IO13); no longer U4.20 (IO12)
- net IO_DAC_BCK: now also U4.25 (IO48); no longer U4.22 (IO14)
- net IO_DAC_DIN: now also U4.24 (IO47); no longer U4.21 (IO13)
- net IO_DAC_LRCK: now also U4.23 (IO21); no longer U4.11 (IO18)
- net IO_VOLUME_DOWN: now also U4.20 (IO12); no longer U4.25 (IO48)
Changed lines of the file:
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@@
+		)
+	)
+	(label "IO_VOLUME_DOWN"
+		(at 72.39 88.9 180)
+		(effects
+			(font
+				(size 1.27 1.27)
+			)
+			(justify right bottom)
 		)
 	)
@@
 		)
 	)
-	(label "IO_VOLUME_DOWN"
-		(at 102.87 93.98 0)
-		(effects
-			(font
-				(size 1.27 1.27)
-			)
-			(justify left bottom)
-		)
-	)
 	(label "IO_VOLUME_UP"
 		(at 113.03 142.24 0)
@@
 		)
 	)
+	(hierarchical_label "IO_DAC_BCK"
+		(shape input)
+		(at 102.87 93.98 0)
+		(effects
+			(font
+				(size 1.27 1.27)
+			)
+			(justify left)
+		)
+	)
+	(hierarchical_label "IO_DAC_LRCK"
+		(shape input)
+		(at 102.87 63.5 0)
+		(effects
+			(font
+				(size 1.27 1.27)
+			)
+			(justify left)
+		)
+	)
+	(hierarchical_label "IO_AUDIO_EN"
+		(shape input)
+		(at 72.39 91.44 180)
+		(effects
+			(font
+				(size 1.27 1.27)
+			)
+			(justify right)
+		)
+	)
+	(hierarchical_label "USB_D+"
+		(shape input)
+		(at 102.87 60.96 0)
+		(effects
+			(font
+				(size 1.27 1.27)
+			)
+			(justify left)
+		)
+	)
+	(hierarchical_label "IO_BAT_V"
+		(shape input)
+		(at 72.39 86.36 180)
+		(effects
+			(font
+				(size 1.27 1.27)
+			)
+			(justify right)
+		)
+	)
+	(hierarchical_label "USB_D-"
+		(shape input)
+		(at 102.87 58.42 0)
+		(effects
+			(font
+				(size 1.27 1.27)
+			)
+			(justify left)
+		)
+	)
+	(hierarchical_label "IO_CHG_STAT1"
+		(shape input)
+		(at 72.39 83.82 180)
+		(effects
+			(font
+				(size 1.27 1.27)
+			)
+			(justify right)
+		)
+	)
 	(hierarchical_label "IO_DAC_DIN"
 		(shape input)
-		(at 72.39 91.44 180)
-		(effects
-			(font
-				(size 1.27 1.27)
-			)
-			(justify right)
-		)
-	)
-	(hierarchical_label "IO_DAC_BCK"
-		(shape input)
-		(at 72.39 93.98 180)
-		(effects
-			(font
-				(size 1.27 1.27)
-			)
-			(justify right)
-		)
-	)
-	(hierarchical_label "IO_DAC_LRCK"
-		(shape input)
-		(at 102.87 55.88 0)
-		(effects
-			(font
-				(size 1.27 1.27)
-			)
-			(justify left)
-		)
-	)
-	(hierarchical_label "USB_D+"
-		(shape input)
-		(at 102.87 60.96 0)
-		(effects
-			(font
-				(size 1.27 1.27)
-			)
-			(justify left)
-		)
-	)
-	(hierarchical_label "IO_BAT_V"
-		(shape input)
-		(at 72.39 86.36 180)
-		(effects
-			(font
-				(size 1.27 1.27)
-			)
-			(justify right)
-		)
-	)
-	(hierarchical_label "USB_D-"
-		(shape input)
-		(at 102.87 58.42 0)
-		(effects
-			(font
-				(size 1.27 1.27)
-			)
-			(justify left)
-		)
-	)
-	(hierarchical_label "IO_AUDIO_EN"
-		(shape input)
-		(at 72.39 88.9 180)
-		(effects
-			(font
-				(size 1.27 1.27)
-			)
-			(justify right)
-		)
-	)
-	(hierarchical_label "IO_CHG_STAT1"
-		(shape input)
-		(at 72.39 83.82 180)
-		(effects
-			(font
-				(size 1.27 1.27)
-			)
-			(justify right)
-		)
-	)
+		(at 102.87 91.44 0)
+		(effects
+			(font
+				(size 1.27 1.27)
+			)
+			(justify left)
+		)
+	)

Commit message: fix sd card pullups
Parts:
- removed TP1: RX, TestPoint:TestPoint_Pad_1.5x1.5mm, symbol Connector:TestPoint
- removed TP2: TX, TestPoint:TestPoint_Pad_1.5x1.5mm, symbol Connector:TestPoint
- added C30: 1µF, Capacitor_SMD:C_0201_0603Metric, symbol Device:C
- added C31: 0.1µF, Capacitor_SMD:C_0201_0603Metric, symbol Device:C
- added R23, R24, R25, R26, R27: 10K, Resistor_SMD:R_0201_0603Metric, symbol Device:R_Small
- C10, C11: value 1uF -> 1µF
Connections:
- net +3V3: now also C30.2
- net GND: now also C30.1, C31.1
- net IO_SD_CMD: now also R27.2
- net IO_SD_DAT0: now also R24.2
- net IO_SD_DAT1: now also R23.2
- net IO_SD_DAT2: now also R25.2
- net IO_SD_DAT3: now also R26.2
- net VSD: now also C31.2, R23.1, R24.1, R25.1, R26.1, R27.1
- no-connect marks 8 -> 10
Other:
- note added: "Screen breakout board contains I2C pullups"
- moved on the sheet: J2, U8

Commit message: switch to stm32, wire audio section
Parts:
- removed C11: 1µF, Capacitor_SMD:C_0201_0603Metric, symbol Device:C
- added C11, C32, C33, C34, C35, C36: 100nF, Capacitor_SMD:C_0402_1005Metric, symbol Device:C_Small
- added C37: 4.7µF, Capacitor_SMD:C_0402_1005Metric, symbol Device:C_Small
- added R22: 10K, Resistor_SMD:R_0402_1005Metric, symbol Device:R_Small
- added U9: STM32F446RETx, Package_QFP:LQFP-64_10x10mm_P0.5mm, symbol MCU_ST_STM32F4:STM32F446RETx
- C10, C30, C31: footprint Capacitor_SMD:C_0201_0603Metric -> Capacitor_SMD:C_0402_1005Metric
- R13, R14, R15, R16, R17, R23, R24, R25, R26, R27: footprint Resistor_SMD:R_0201_0603Metric -> Resistor_SMD:R_0402_1005Metric
Connections:
- net +3V3: now also S2.1, C11.1, C32.1, C33.1, C34.1, C35.1, C36.1, C37.1, U9.1 (VBAT), U9.13 (VDDA), U9.19 (VDD), U9.32 (VDD), U9.48 (VDD), U9.64 (VDD); no longer R15.1
- net GND: now also R15.1, C11.2, C32.2, C33.2, C34.2, C35.2, C36.2, C37.2, R22.1, U9.12 (VSSA), U9.18 (VSS), U9.28 (PB2), U9.31 (VSS), U9.47 (VSS), U9.63 (VSS); no longer S2.2
- net IO_BOOT: now also S2.2, U9.60 (BOOT0); no longer S2.1
- net IO_DAC_BCK: now also U9.38 (PC7)
- net IO_DAC_DIN: now also U9.9 (PC1)
- net IO_DAC_LRCK: now also U9.62 (PB9)
- net IO_EN: no longer C10.1, R13.2, S1.1
- net IO_SD_CLK: now also U9.53 (PC12)
- net IO_SD_CMD: now also U9.54 (PD2)
- net IO_SD_DAT0: now also U9.39 (PC8)
- net IO_SD_DAT1: no longer J2.8 (DAT1), R23.2
- net IO_SD_DAT2: no longer J2.1 (DAT2), R25.2
- net IO_SD_DAT3: no longer J2.2 (CD/DAT3), R26.2
- net IO_SD_EN: now also R22.2, U9.29 (PB10)
- net USB_D+: now also U9.45 (PA12)
- net USB_D-: now also U9.44 (PA11)
- new net: J2.2 (CD/DAT3), R26.2
- new net: J2.1 (DAT2), R25.2
- new net: J2.8 (DAT1), R23.2
- new net IO_RESET: C10.1, R13.2, S1.1, U9.7 (NRST)
Other:
- moved on the sheet: C10, R13, R14, R15, R16, R17, R23, R25, R26, S1, S2, S3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

Commit message: add clock
Parts:
- added C38, C39: 22pF, Capacitor_SMD:C_0402_1005Metric, symbol Device:C_Small
- added Y1: X50328MSB2GI, Crystal:Crystal_SMD_5032-2Pin_5.0x3.2mm, symbol Device:Crystal
Connections:
- net GND: now also C38.2, C39.2
- net OSC-: now reaches U9.5 (PH0)
- net OSC-: now also C38.1, Y1.1
- net OSC+: now reaches U9.6 (PH1)
- net OSC+: now also C39.1, Y1.2
Other:
- moved on the sheet: C11, C32, C33, C34, C35, C36, C37, U9
