File: mcu.kicad_sch (KiCad schematic)
At the start: 33 parts, among them J2 DM3CS-SF, J4 SCREEN, U4 ESP32-S3-WROOM-1U-N16R8, U8 SiP32431DR3, U9 STM32F446RETx, Y1 X50328MSB2GI

Commit message: some fixes
Parts:
- removed R14: 10K, Resistor_SMD:R_0402_1005Metric, symbol Device:R_Small
- removed U4: ESP32-S3-WROOM-1U-N16R8, esp32:XCVR_ESP32-S3-WROOM-1U-N16R8, symbol ESP32-S3-WROOM-1U-N16R8:ESP32-S3-WROOM-1U-N16R8
Connections:
- net IO_BAT_V: now also U9.52 (PC11)
- net IO_CHG_STAT1: now also U9.46 (PA13)
- net IO_CHG_STAT2: now also U9.51 (PC10)
- net IO_I2C_SCL: now also U9.58 (PB6)
- net IO_I2C_SDA: now also U9.59 (PB7)
- net IO_VOLUME_DOWN: now also U9.57 (PB5)
- net IO_VOLUME_UP: now also U9.56 (PB4)
- no-connect marks 10 -> 3

Commit message: fill more parts
Parts:
- Y1: LCSC Part # (none) -> C115962; Part # (none) -> X50328MSB2GI
Connections:
- net IO_BAT_V: now also U9.23 (PA7); no longer U9.52 (PC11)
- net IO_CHG_STAT1: now also U9.24 (PC4); no longer U9.46 (PA13)
- net IO_VOLUME_UP: no longer U9.56 (PB4)
- net IO_PLAY_POWER: now reaches U9.14 (PA0)
- no-connect marks 3 -> 8
Changed lines of the file:
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@@
 	)
 	(no_connect
+		(at 101.6 80.01)
+	)
+	(no_connect
+		(at 101.6 82.55)
+	)
+	(no_connect
+		(at 101.6 97.79)
+	)
+	(no_connect
 		(at 82.55 186.69)
 	)
 	(no_connect
+		(at 101.6 77.47)
+	)
+	(no_connect
 		(at 200.66 36.83)
 	)
@@
 		(at 82.55 163.83)
 	)
+	(no_connect
+		(at 101.6 95.25)
+	)
 	(wire
 		(pts
@@
 		)
 	)
-	(label "IO_VOLUME_UP"
-		(at 101.6 97.79 0)
+	(label "IO_SD_DAT0"
+		(at 173.99 39.37 180)
 		(effects
 			(font
 				(size 1.27 1.27)
 			)
-			(justify left bottom)
+			(justify right bottom)
 		)
 	)
-	(label "IO_SD_DAT0"
-		(at 173.99 39.37 180)
+	(label "IO_SD_CMD"
+		(at 60.96 62.23 180)
 		(effects
 			(font
@@
 		)
 	)
-	(label "IO_SD_CMD"
-		(at 60.96 62.23 180)
+	(label "IO_PLAY_POWER"
+		(at 101.6 44.45 0)
 		(effects
 			(font
 				(size 1.27 1.27)
 			)
-			(justify right bottom)
+			(justify left bottom)
 		)
 	)
@@
 	)
 	(label "IO_VOLUME_UP"
+		(at 118.11 97.79 0)
+		(effects
+			(font
+				(size 1.27 1.27)
+			)
+			(justify left bottom)
+		)
+	)
+	(label "IO_VOLUME_UP"
 		(at 110.49 161.29 0)
 		(effects
@@
 		)
 	)
-	(hierarchical_label "IO_CHG_STAT1"
+	(hierarchical_label "IO_DAC_LRCK"
 		(shape input)
-		(at 101.6 77.47 0)
+		(at 101.6 110.49 0)
 		(effects
 			(font
@@
 		)
 	)
-	(hierarchical_label "IO_DAC_LRCK"
+	(hierarchical_label "IO_BAT_V"
 		(shape input)
-		(at 101.6 110.49 0)
+		(at 101.6 62.23 0)
 		(effects
 			(font
@@
 		)
 	)
-	(hierarchical_label "USB_D+"
+	(hierarchical_label "IO_CHG_STAT1"
 		(shape input)
-		(at 101.6 74.93 0)
+		(at 60.96 77.47 180)
 		(effects
 			(font
 				(size 1.27 1.27)
 			)
-			(justify left)
+			(justify right)
 		)
 	)
-	(hierarchical_label "IO_BAT_V"
+	(hierarchical_label "USB_D+"
 		(shape input)
-		(at 60.96 95.25 180)
+		(at 101.6 74.93 0)
 		(effects
 			(font
 				(size 1.27 1.27)
 			)
-			(justify right)
+			(justify left)
 		)
 	)
@@
 			)
 		)
-		(property "LCSC Part #" ""
+		(property "LCSC Part #" "C115962"
 			(at 27.94 57.15 0)
 			(hide yes)
@@
 			)
 		)
-		(property "Part #" ""
+		(property "Part #" "X50328MSB2GI"
 			(at 27.94 57.15 0)
 			(hide yes)

Commit message: label sections
Other:
- note added: "Buttons"
- note added: "Micro SD"
- moved on the sheet: C11, C30, C31, C32, C33, C34, C35, C36, C37, C38, C39, J2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
